File: regulateur.brd (EAGLE design)
At the start: 41.9 x 29.2 mm, 16 parts, among them U1 LT1372CS8PBF

Commit message: Add files via upload
change package R2 , R1 , R3 , C3
Parts:
- removed D2: GSOT05C-E3-08, diode:SOT23
- C3: device resistor:C0402 -> resistor:C1206
- R1, R2, R3: device resistor:R0402 -> resistor:R1206
- moved R3 1.72 mm to (33.8, 30.9)
- moved C3 1.15 mm to (33.8, 34.2)
- moved R1 0.18 mm to (33.8, 24.9)
Connections:
- net GND: no longer D2.1
- net N$6: no longer D2.2
Routing:
- net N$6: track 84.7 -> 78.8 mm
- net N$1: track 6.06 -> 3.90 mm
- net N$2: track 15.7 -> 14.4 mm

Commit message: Add files via upload
Parts:
- R1: value 12.76K -> 10K
- R2: value 37.24K -> 31.6K
- R3: value 5K -> 5.1K
Changed lines of the file:
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@@
 <element name="C5" library="resistor" package="CT7343" value="22uF" x="24.765" y="26.67" rot="R180"/>
 <element name="C1" library="resistor" package="CT7343" value="22uF" x="13.97" y="26.67" rot="R180"/>
-<element name="R1" library="resistor" package="R1206" value="12.76K" x="33.782" y="24.892"/>
-<element name="R2" library="resistor" package="R1206" value="37.24K" x="33.655" y="21.59" rot="R180"/>
-<element name="R3" library="resistor" package="R1206" value="5K" x="33.782" y="30.9245"/>
+<element name="R1" library="resistor" package="R1206" value="10K" x="33.782" y="24.892"/>
+<element name="R2" library="resistor" package="R1206" value="31.6K" x="33.655" y="21.59" rot="R180"/>
+<element name="R3" library="resistor" package="R1206" value="5.1K" x="33.782" y="30.9245"/>
 <element name="C2" library="resistor" package="C1206" value="10nF" x="39.37" y="33.655" rot="R180"/>
 <element name="C3" library="resistor" package="C1206" value="200pF" x="33.782" y="34.163" rot="R180"/>

Commit message: Add files via upload
Parts:
- renumbered PAD1 to VOUT, PAD2 to VIN, PAD3 to GND_IN, PAD4 to GND_OUT
Changed lines of the file:
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@@
 <layer number="25" name="tNames" color="7" fill="1" visible="yes" active="yes"/>
 <layer number="26" name="bNames" color="7" fill="1" visible="no" active="yes"/>
-<layer number="27" name="tValues" color="7" fill="1" visible="yes" active="yes"/>
+<layer number="27" name="tValues" color="7" fill="1" visible="no" active="yes"/>
 <layer number="28" name="bValues" color="7" fill="1" visible="no" active="yes"/>
 <layer number="29" name="tStop" color="7" fill="3" visible="no" active="yes"/>
@@
 <layer number="39" name="tKeepout" color="4" fill="11" visible="no" active="yes"/>
 <layer number="40" name="bKeepout" color="1" fill="11" visible="no" active="yes"/>
-<layer number="41" name="tRestrict" color="4" fill="10" visible="yes" active="yes"/>
+<layer number="41" name="tRestrict" color="4" fill="10" visible="no" active="yes"/>
 <layer number="42" name="bRestrict" color="1" fill="10" visible="no" active="yes"/>
 <layer number="43" name="vRestrict" color="2" fill="10" visible="no" active="yes"/>
@@
 <element name="C2" library="resistor" package="C1206" value="10nF" x="39.37" y="33.655" rot="R180"/>
 <element name="C3" library="resistor" package="C1206" value="200pF" x="33.782" y="34.163" rot="R180"/>
-<element name="PAD1" library="wirepad" package="3,81/1,3" value="OUT" x="11.43" y="38.735"/>
-<element name="PAD2" library="wirepad" package="3,81/1,3" value="IN" x="45.72" y="38.735"/>
-<element name="PAD3" library="wirepad" package="3,81/1,3" value="IN_GND" x="45.72" y="21.59"/>
-<element name="PAD4" library="wirepad" package="3,81/1,3" value="OUT_GND" x="11.43" y="21.59"/>
+<element name="VOUT" library="wirepad" package="3,81/1,3" value="OUT" x="11.43" y="38.735"/>
+<element name="VIN" library="wirepad" package="3,81/1,3" value="IN" x="45.72" y="38.735"/>
+<element name="GND_IN" library="wirepad" package="3,81/1,3" value="IN_GND" x="45.72" y="21.59"/>
+<element name="GND_OUT" library="wirepad" package="3,81/1,3" value="OUT_GND" x="11.43" y="21.59"/>
 </elements>
 <signals>
@@
 <contactref element="C1" pad="+"/>
 <contactref element="R2" pad="2"/>
-<contactref element="PAD1" pad="1"/>
+<contactref element="VOUT" pad="1"/>
 <wire x1="22.5" y1="21.75" x2="22.565" y2="21.59" width="0.4032" layer="1"/>
 <wire x1="30.508" y1="23.095" x2="31.7236375" y2="21.5912375" width="0.6096" layer="1"/>
@@
 <contactref element="R1" pad="1"/>
 <contactref element="R3" pad="1"/>
-<contactref element="PAD3" pad="1"/>
-<contactref element="PAD4" pad="1"/>
+<contactref element="GND_IN" pad="1"/>
+<contactref element="GND_OUT" pad="1"/>
 <wire x1="43.128859375" y1="27.8466625" x2="43.1120625" y2="26.813340625" width="0.6096" layer="1"/>
 <wire x1="43.1120625" y1="26.813340625" x2="43.1038" y2="26.67" width="0.4032" layer="1"/>
@@
 <contactref element="U1" pad="5"/>
 <contactref element="L1" pad="3"/>
-<contactref element="PAD2" pad="1"/>
+<contactref element="VIN" pad="1"/>
 <wire x1="40.5" y1="43.187834375" x2="25.75" y2="43.187834375" width="0.8128" layer="1"/>
 <wire x1="40.5" y1="40.25" x2="40.5" y2="43.187834375" width="0.8128" layer="1"/>

Commit message: Add files via upload
Parts:
- R1: value 10K -> 12.76K; device resistor:R1206 -> resistor:M1206
- R2: value 31.6K -> 37.24K; device resistor:R1206 -> resistor:M1206
- R3: value 5.1K -> 5K; device resistor:R1206 -> resistor:M1206
- U1: value LT1372CS8PBF -> LT1372
- moved C3 0.77 mm to (33.7, 34.9)
- moved R3 0.46 mm to (33.7, 30.5)
- moved R1 0.18 mm to (33.7, 24.8)
- renumbered VIN to IN, VOUT to OUT
Routing:
- net N$4: track 42.0 -> 53.8 mm
- net N$6: track 78.8 -> 80.4 mm
- net N$2: track 14.4 -> 13.0 mm
- net N$1: track 3.90 -> 5.16 mm
- net GND: track 98.3 -> 99.5 mm
- added copper zone on layer 16, net GND
