File: regulateur.sch (EAGLE design)
At the start: 16 parts, among them U1 LT1372CS8PBF

Commit message: Add files via upload
change package R2 , R1 , R3 , C3
Parts:
- removed D2: GSOT05C-E3-08, diode:BAS40-06
- C3: device resistor:C-EUC0402 -> resistor:C-EUC1206
- R1, R2, R3: device resistor:R-EU_R0402 -> resistor:R-EU_R1206
Connections:
- net GND: no longer D2.K1
- net N$6: no longer D2.K2
Changed lines of the file:
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@@
 <grid distance="0.1" unitdist="inch" unit="inch" style="lines" multiple="1" display="no" altdistance="0.01" altunitdist="inch" altunit="inch"/>
 <layers>
-<layer number="1" name="Top" color="4" fill="1" visible="no" active="no"/>
-<layer number="16" name="Bottom" color="1" fill="1" visible="no" active="no"/>
-<layer number="17" name="Pads" color="2" fill="1" visible="no" active="no"/>
-<layer number="18" name="Vias" color="2" fill="1" visible="no" active="no"/>
-<layer number="19" name="Unrouted" color="6" fill="1" visible="no" active="no"/>
-<layer number="20" name="Dimension" color="15" fill="1" visible="no" active="no"/>
-<layer number="21" name="tPlace" color="7" fill="1" visible="no" active="no"/>
-<layer number="22" name="bPlace" color="7" fill="1" visible="no" active="no"/>
-<layer number="23" name="tOrigins" color="15" fill="1" visible="no" active="no"/>
-<layer number="24" name="bOrigins" color="15" fill="1" visible="no" active="no"/>
-<layer number="25" name="tNames" color="7" fill="1" visible="no" active="no"/>
-<layer number="26" name="bNames" color="7" fill="1" visible="no" active="no"/>
-<layer number="27" name="tValues" color="7" fill="1" visible="no" active="no"/>
-<layer number="28" name="bValues" color="7" fill="1" visible="no" active="no"/>
+<layer number="1" name="Top" color="4" fill="1" visible="yes" active="no"/>
+<layer number="16" name="Bottom" color="1" fill="1" visible="yes" active="no"/>
+<layer number="17" name="Pads" color="2" fill="1" visible="yes" active="no"/>
+<layer number="18" name="Vias" color="2" fill="1" visible="yes" active="no"/>
+<layer number="19" name="Unrouted" color="6" fill="1" visible="yes" active="no"/>
+<layer number="20" name="Dimension" color="15" fill="1" visible="yes" active="no"/>
+<layer number="21" name="tPlace" color="7" fill="1" visible="yes" active="no"/>
+<layer number="22" name="bPlace" color="7" fill="1" visible="yes" active="no"/>
+<layer number="23" name="tOrigins" color="15" fill="1" visible="yes" active="no"/>
+<layer number="24" name="bOrigins" color="15" fill="1" visible="yes" active="no"/>
+<layer number="25" name="tNames" color="7" fill="1" visible="yes" active="no"/>
+<layer number="26" name="bNames" color="7" fill="1" visible="yes" active="no"/>
+<layer number="27" name="tValues" color="7" fill="1" visible="yes" active="no"/>
+<layer number="28" name="bValues" color="7" fill="1" visible="yes" active="no"/>
 <layer number="29" name="tStop" color="7" fill="3" visible="no" active="no"/>
 <layer number="30" name="bStop" color="7" fill="6" visible="no" active="no"/>
@@
 <layer number="35" name="tGlue" color="7" fill="4" visible="no" active="no"/>
 <layer number="36" name="bGlue" color="7" fill="5" visible="no" active="no"/>
-<layer number="37" name="tTest" color="7" fill="1" visible="no" active="no"/>
-<layer number="38" name="bTest" color="7" fill="1" visible="no" active="no"/>
+<layer number="37" name="tTest" color="7" fill="1" visible="yes" active="no"/>
+<layer number="38" name="bTest" color="7" fill="1" visible="yes" active="no"/>
 <layer number="39" name="tKeepout" color="4" fill="11" visible="no" active="no"/>
 <layer number="40" name="bKeepout" color="1" fill="11" visible="no" active="no"/>
@@
 <layer number="44" name="Drills" color="7" fill="1" visible="no" active="no"/>
 <layer number="45" name="Holes" color="7" fill="1" visible="no" active="no"/>
-<layer number="46" name="Milling" color="3" fill="1" visible="no" active="no"/>
-<layer number="47" name="Measures" color="7" fill="1" visible="no" active="no"/>
-<layer number="48" name="Document" color="7" fill="1" visible="no" active="no"/>
-<layer number="49" name="Reference" color="7" fill="1" visible="no" active="no"/>
-<layer number="50" name="dxf" color="7" fill="1" visible="no" active="no"/>
-<layer number="51" name="tDocu" color="7" fill="1" visible="no" active="no"/>
-<layer number="52" name="bDocu" color="7" fill="1" visible="no" active="no"/>
-<layer number="53" name="tPadExt" color="7" fill="1" visible="no" active="no"/>
-<layer number="54" name="bPadExt" color="1" fill="1" visible="no" active="no"/>
+<layer number="46" name="Milling" color="3" fill="1" visible="yes" active="no"/>
+<layer number="47" name="Measures" color="7" fill="1" visible="yes" active="no"/>
+<layer number="48" name="Document" color="7" fill="1" visible="yes" active="no"/>
+<layer number="49" name="Reference" color="7" fill="1" visible="yes" active="no"/>
+<layer number="50" name="dxf" color="7" fill="1" visible="yes" active="no"/>
+<layer number="51" name="tDocu" color="7" fill="1" visible="yes" active="no"/>
+<layer number="52" name="bDocu" color="7" fill="1" visible="yes" active="no"/>
+<layer number="53" name="tPadExt" color="7" fill="1" visible="yes" active="no"/>
+<layer number="54" name="bPadExt" color="1" fill="1" visible="yes" active="no"/>
 <layer number="90" name="Modules" color="5" fill="1" visible="yes" active="yes"/>
 <layer number="91" name="Nets" color="2" fill="1" visible="yes" active="yes"/>
@@
 <part name="C5" library="resistor" deviceset="CPOL-EU" device="CT7343" value="22uF"/>
 <part name="C1" library="resistor" deviceset="CPOL-EU" device="CT7343" value="22uF"/>
-<part name="R1" library="resistor" deviceset="R-EU_" device="R0402" value="12.76K"/>
-<part name="R2" library="resistor" deviceset="R-EU_" device="R0402" value="37.24K"/>
-<part name="R3" library="resistor" deviceset="R-EU_" device="R0402" value="5K"/>
+<part name="R1" library="resistor" deviceset="R-EU_" device="R1206" value="12.76K"/>
+<part name="R2" library="resistor" deviceset="R-EU_" device="R1206" value="37.24K"/>
+<part name="R3" library="resistor" deviceset="R-EU_" device="R1206" value="5K"/>
 <part name="C2" library="resistor" deviceset="C-EU" device="C1206" value="10nF"/>
-<part name="C3" library="resistor" deviceset="C-EU" device="C0402" value="200pF"/>
+<part name="C3" library="resistor" deviceset="C-EU" device="C1206" value="200pF"/>
 <part name="GND1" library="supply1" deviceset="GND" device=""/>
 <part name="GND2" library="supply1" deviceset="GND" device=""/>
@@
 <part name="PAD3" library="wirepad" deviceset="3,81/1,3" device="" value="IN_GND"/>
 <part name="PAD4" library="wirepad" deviceset="3,81/1,3" device="" value="OUT_GND"/>
-<part name="D2" library="diode" deviceset="BAS40-06" device="" value="GSOT05C-E3-08"/>
 <part name="GND6" library="supply1" deviceset="GND" device=""/>
 </parts>
@@
 <instance part="PAD3" gate="1" x="-17.78" y="60.96"/>
 <instance part="PAD4" gate="1" x="144.78" y="33.02" rot="R180"/>
-<instance part="D2" gate="G$1" x="132.08" y="48.26" rot="R90"/>
 <instance part="GND6" gate="1" x="132.08" y="25.4"/>
 </instances>
@@
 <junction x="121.92" y="60.96"/>
 <pinref part="PAD1" gate="1" pin="P"/>
-<wire x1="121.92" y1="63.5" x2="132.08" y2="63.5" width="0.1524" layer="91"/>
 <junction x="121.92" y="63.5"/>
 <junction x="142.24" y="63.5"/>
-<pinref part="D2" gate="G$1" pin="K2"/>
-<wire x1="132.08" y1="63.5" x2="142.24" y2="63.5" width="0.1524" layer="91"/>
-<wire x1="132.08" y1="53.34" x2="132.08" y2="63.5" width="0.1524" layer="91"/>
-<junction x="132.08" y="63.5"/>
-<junction x="132.08" y="53.34"/>
+<wire x1="121.92" y1="63.5" x2="142.24" y2="63.5" width="0.1524" layer="91"/>
 </segment>
 </net>
@@
 <junction x="142.24" y="33.02"/>
 <wire x1="132.08" y1="33.02" x2="142.24" y2="33.02" width="0.1524" layer="91"/>
-<pinref part="D2" gate="G$1" pin="K1"/>
-<junction x="132.08" y="43.18"/>
-<wire x1="132.08" y1="43.18" x2="132.08" y2="33.02" width="0.1524" layer="91"/>
 <pinref part="GND6" gate="1" pin="GND"/>
 <wire x1="132.08" y1="33.02" x2="132.08" y2="27.94" width="0.1524" layer="91"/>
-<junction x="132.08" y="33.02"/>
 <junction x="132.08" y="27.94"/>
 </segment>

Commit message: Add files via upload
Parts:
- R1: value 12.76K -> 10K
- R2: value 37.24K -> 31.6K
- R3: value 5K -> 5.1K
Changed lines of the file:
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@@
 <grid distance="0.1" unitdist="inch" unit="inch" style="lines" multiple="1" display="no" altdistance="0.01" altunitdist="inch" altunit="inch"/>
 <layers>
-<layer number="1" name="Top" color="4" fill="1" visible="yes" active="no"/>
-<layer number="16" name="Bottom" color="1" fill="1" visible="yes" active="no"/>
-<layer number="17" name="Pads" color="2" fill="1" visible="yes" active="no"/>
-<layer number="18" name="Vias" color="2" fill="1" visible="yes" active="no"/>
-<layer number="19" name="Unrouted" color="6" fill="1" visible="yes" active="no"/>
-<layer number="20" name="Dimension" color="15" fill="1" visible="yes" active="no"/>
-<layer number="21" name="tPlace" color="7" fill="1" visible="yes" active="no"/>
-<layer number="22" name="bPlace" color="7" fill="1" visible="yes" active="no"/>
-<layer number="23" name="tOrigins" color="15" fill="1" visible="yes" active="no"/>
-<layer number="24" name="bOrigins" color="15" fill="1" visible="yes" active="no"/>
-<layer number="25" name="tNames" color="7" fill="1" visible="yes" active="no"/>
-<layer number="26" name="bNames" color="7" fill="1" visible="yes" active="no"/>
-<layer number="27" name="tValues" color="7" fill="1" visible="yes" active="no"/>
-<layer number="28" name="bValues" color="7" fill="1" visible="yes" active="no"/>
+<layer number="1" name="Top" color="4" fill="1" visible="no" active="no"/>
+<layer number="16" name="Bottom" color="1" fill="1" visible="no" active="no"/>
+<layer number="17" name="Pads" color="2" fill="1" visible="no" active="no"/>
+<layer number="18" name="Vias" color="2" fill="1" visible="no" active="no"/>
+<layer number="19" name="Unrouted" color="6" fill="1" visible="no" active="no"/>
+<layer number="20" name="Dimension" color="15" fill="1" visible="no" active="no"/>
+<layer number="21" name="tPlace" color="7" fill="1" visible="no" active="no"/>
+<layer number="22" name="bPlace" color="7" fill="1" visible="no" active="no"/>
+<layer number="23" name="tOrigins" color="15" fill="1" visible="no" active="no"/>
+<layer number="24" name="bOrigins" color="15" fill="1" visible="no" active="no"/>
+<layer number="25" name="tNames" color="7" fill="1" visible="no" active="no"/>
+<layer number="26" name="bNames" color="7" fill="1" visible="no" active="no"/>
+<layer number="27" name="tValues" color="7" fill="1" visible="no" active="no"/>
+<layer number="28" name="bValues" color="7" fill="1" visible="no" active="no"/>
 <layer number="29" name="tStop" color="7" fill="3" visible="no" active="no"/>
 <layer number="30" name="bStop" color="7" fill="6" visible="no" active="no"/>
@@
 <layer number="35" name="tGlue" color="7" fill="4" visible="no" active="no"/>
 <layer number="36" name="bGlue" color="7" fill="5" visible="no" active="no"/>
-<layer number="37" name="tTest" color="7" fill="1" visible="yes" active="no"/>
-<layer number="38" name="bTest" color="7" fill="1" visible="yes" active="no"/>
+<layer number="37" name="tTest" color="7" fill="1" visible="no" active="no"/>
+<layer number="38" name="bTest" color="7" fill="1" visible="no" active="no"/>
 <layer number="39" name="tKeepout" color="4" fill="11" visible="no" active="no"/>
 <layer number="40" name="bKeepout" color="1" fill="11" visible="no" active="no"/>
@@
 <layer number="44" name="Drills" color="7" fill="1" visible="no" active="no"/>
 <layer number="45" name="Holes" color="7" fill="1" visible="no" active="no"/>
-<layer number="46" name="Milling" color="3" fill="1" visible="yes" active="no"/>
-<layer number="47" name="Measures" color="7" fill="1" visible="yes" active="no"/>
-<layer number="48" name="Document" color="7" fill="1" visible="yes" active="no"/>
-<layer number="49" name="Reference" color="7" fill="1" visible="yes" active="no"/>
-<layer number="50" name="dxf" color="7" fill="1" visible="yes" active="no"/>
-<layer number="51" name="tDocu" color="7" fill="1" visible="yes" active="no"/>
-<layer number="52" name="bDocu" color="7" fill="1" visible="yes" active="no"/>
-<layer number="53" name="tPadExt" color="7" fill="1" visible="yes" active="no"/>
-<layer number="54" name="bPadExt" color="1" fill="1" visible="yes" active="no"/>
+<layer number="46" name="Milling" color="3" fill="1" visible="no" active="no"/>
+<layer number="47" name="Measures" color="7" fill="1" visible="no" active="no"/>
+<layer number="48" name="Document" color="7" fill="1" visible="no" active="no"/>
+<layer number="49" name="Reference" color="7" fill="1" visible="no" active="no"/>
+<layer number="50" name="dxf" color="7" fill="1" visible="no" active="no"/>
+<layer number="51" name="tDocu" color="7" fill="1" visible="no" active="no"/>
+<layer number="52" name="bDocu" color="7" fill="1" visible="no" active="no"/>
+<layer number="53" name="tPadExt" color="7" fill="1" visible="no" active="no"/>
+<layer number="54" name="bPadExt" color="1" fill="1" visible="no" active="no"/>
 <layer number="90" name="Modules" color="5" fill="1" visible="yes" active="yes"/>
 <layer number="91" name="Nets" color="2" fill="1" visible="yes" active="yes"/>
@@
 <part name="C5" library="resistor" deviceset="CPOL-EU" device="CT7343" value="22uF"/>
 <part name="C1" library="resistor" deviceset="CPOL-EU" device="CT7343" value="22uF"/>
-<part name="R1" library="resistor" deviceset="R-EU_" device="R1206" value="12.76K"/>
-<part name="R2" library="resistor" deviceset="R-EU_" device="R1206" value="37.24K"/>
-<part name="R3" library="resistor" deviceset="R-EU_" device="R1206" value="5K"/>
+<part name="R1" library="resistor" deviceset="R-EU_" device="R1206" value="10K"/>
+<part name="R2" library="resistor" deviceset="R-EU_" device="R1206" value="31.6K"/>
+<part name="R3" library="resistor" deviceset="R-EU_" device="R1206" value="5.1K"/>
 <part name="C2" library="resistor" deviceset="C-EU" device="C1206" value="10nF"/>
 <part name="C3" library="resistor" deviceset="C-EU" device="C1206" value="200pF"/>

Commit message: Add files via upload
Parts:
- renumbered PAD1 to VOUT, PAD2 to VIN, PAD3 to GND_IN, PAD4 to GND_OUT
Changed lines of the file:
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@@
 <part name="P+1" library="supply1" deviceset="VCC" device=""/>
 <part name="GND5" library="supply1" deviceset="GND" device=""/>
-<part name="PAD1" library="wirepad" deviceset="3,81/1,3" device="" value="OUT"/>
-<part name="PAD2" library="wirepad" deviceset="3,81/1,3" device="" value="IN"/>
-<part name="PAD3" library="wirepad" deviceset="3,81/1,3" device="" value="IN_GND"/>
-<part name="PAD4" library="wirepad" deviceset="3,81/1,3" device="" value="OUT_GND"/>
+<part name="VOUT" library="wirepad" deviceset="3,81/1,3" device="" value="OUT"/>
+<part name="VIN" library="wirepad" deviceset="3,81/1,3" device="" value="IN"/>
+<part name="GND_IN" library="wirepad" deviceset="3,81/1,3" device="" value="IN_GND"/>
+<part name="GND_OUT" library="wirepad" deviceset="3,81/1,3" device="" value="OUT_GND"/>
 <part name="GND6" library="supply1" deviceset="GND" device=""/>
 </parts>
@@
 <instance part="P+1" gate="VCC" x="-2.54" y="88.9"/>
 <instance part="GND5" gate="1" x="22.86" y="38.1"/>
-<instance part="PAD1" gate="1" x="144.78" y="63.5" rot="R180"/>
-<instance part="PAD2" gate="1" x="-17.78" y="81.28"/>
-<instance part="PAD3" gate="1" x="-17.78" y="60.96"/>
-<instance part="PAD4" gate="1" x="144.78" y="33.02" rot="R180"/>
+<instance part="VOUT" gate="1" x="144.78" y="63.5" rot="R180"/>
+<instance part="VIN" gate="1" x="-17.78" y="81.28"/>
+<instance part="GND_IN" gate="1" x="-17.78" y="60.96"/>
+<instance part="GND_OUT" gate="1" x="144.78" y="33.02" rot="R180"/>
 <instance part="GND6" gate="1" x="132.08" y="25.4"/>
 </instances>
@@
 <junction x="109.22" y="58.42"/>
 <junction x="121.92" y="60.96"/>
-<pinref part="PAD1" gate="1" pin="P"/>
+<pinref part="VOUT" gate="1" pin="P"/>
 <junction x="121.92" y="63.5"/>
 <junction x="142.24" y="63.5"/>
@@
 <junction x="-2.54" y="68.58"/>
 <junction x="-2.54" y="60.96"/>
-<pinref part="PAD3" gate="1" pin="P"/>
+<pinref part="GND_IN" gate="1" pin="P"/>
 <wire x1="-15.24" y1="60.96" x2="-2.54" y2="60.96" width="0.1524" layer="91"/>
 <junction x="-15.24" y="60.96"/>
@@
 </segment>
 <segment>
-<pinref part="PAD4" gate="1" pin="P"/>
+<pinref part="GND_OUT" gate="1" pin="P"/>
 <junction x="142.24" y="33.02"/>
 <wire x1="132.08" y1="33.02" x2="142.24" y2="33.02" width="0.1524" layer="91"/>
@@
 <junction x="20.32" y="81.28"/>
 <junction x="53.34" y="81.28"/>
-<pinref part="PAD2" gate="1" pin="P"/>
+<pinref part="VIN" gate="1" pin="P"/>
 <wire x1="-15.24" y1="81.28" x2="-2.54" y2="81.28" width="0.1524" layer="91"/>
 <junction x="-15.24" y="81.28"/>

Commit message: Add files via upload
Parts:
- R1: value 10K -> 12.76K; device resistor:R-EU_R1206 -> resistor:R-EU_M1206
- R2: value 31.6K -> 37.24K; device resistor:R-EU_R1206 -> resistor:R-EU_M1206
- R3: value 5.1K -> 5K; device resistor:R-EU_R1206 -> resistor:R-EU_M1206
- U1: value LT1372CS8PBF -> LT1372
- renumbered VIN to IN, VOUT to OUT
Other:
- note added: "R1 = 10K R2 = 31.6K Vout = 5.1v"
- note added: "R1 = 12.7K R2 = 39K Vout = 5.1v"
Changed lines of the file:
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@@
 <?xml version="1.0" encoding="utf-8"?>
 <!DOCTYPE eagle SYSTEM "eagle.dtd">
-<eagle version="7.6.0">
+<eagle version="7.5.0">
 <drawing>
 <settings>
@@
 </classes>
 <parts>
-<part name="U1" library="LTC_By_element14_Batch_1" deviceset="LT1372CS8PBF" device=""/>
+<part name="U1" library="LTC_By_element14_Batch_1" deviceset="LT1372CS8PBF" device="" value="LT1372"/>
 <part name="L1" library="WE-DD" deviceset="WE-DD" device="_1260/1280/1210_CROSSED" technology="-744871220" value="22uH"/>
 <part name="D1" library="diode" deviceset="MBRS130LT3" device=""/>
@@
 <part name="C5" library="resistor" deviceset="CPOL-EU" device="CT7343" value="22uF"/>
 <part name="C1" library="resistor" deviceset="CPOL-EU" device="CT7343" value="22uF"/>
-<part name="R1" library="resistor" deviceset="R-EU_" device="R1206" value="10K"/>
-<part name="R2" library="resistor" deviceset="R-EU_" device="R1206" value="31.6K"/>
-<part name="R3" library="resistor" deviceset="R-EU_" device="R1206" value="5.1K"/>
+<part name="R1" library="resistor" deviceset="R-EU_" device="M1206" value="12.76K"/>
+<part name="R2" library="resistor" deviceset="R-EU_" device="M1206" value="37.24K"/>
+<part name="R3" library="resistor" deviceset="R-EU_" device="M1206" value="5K"/>
 <part name="C2" library="resistor" deviceset="C-EU" device="C1206" value="10nF"/>
 <part name="C3" library="resistor" deviceset="C-EU" device="C1206" value="200pF"/>
@@
 <part name="P+1" library="supply1" deviceset="VCC" device=""/>
 <part name="GND5" library="supply1" deviceset="GND" device=""/>
-<part name="VOUT" library="wirepad" deviceset="3,81/1,3" device="" value="OUT"/>
-<part name="VIN" library="wirepad" deviceset="3,81/1,3" device="" value="IN"/>
+<part name="OUT" library="wirepad" deviceset="3,81/1,3" device="" value="OUT"/>
+<part name="IN" library="wirepad" deviceset="3,81/1,3" device="" value="IN"/>
 <part name="GND_IN" library="wirepad" deviceset="3,81/1,3" device="" value="IN_GND"/>
 <part name="GND_OUT" library="wirepad" deviceset="3,81/1,3" device="" value="OUT_GND"/>
@@
 <sheet>
 <plain>
+<text x="68.58" y="20.32" size="1.778" layer="91">R1 = 12.7K  R2 = 39K   Vout = 5.1v</text>
+<text x="68.58" y="15.24" size="1.778" layer="91">R1 = 10K  R2 = 31.6K  Vout = 5.1v</text>
 </plain>
 <instances>
@@
 <instance part="P+1" gate="VCC" x="-2.54" y="88.9"/>
 <instance part="GND5" gate="1" x="22.86" y="38.1"/>
-<instance part="VOUT" gate="1" x="144.78" y="63.5" rot="R180"/>
-<instance part="VIN" gate="1" x="-17.78" y="81.28"/>
+<instance part="OUT" gate="1" x="144.78" y="63.5" rot="R180"/>
+<instance part="IN" gate="1" x="-17.78" y="81.28"/>
 <instance part="GND_IN" gate="1" x="-17.78" y="60.96"/>
 <instance part="GND_OUT" gate="1" x="144.78" y="33.02" rot="R180"/>
@@
 <junction x="109.22" y="58.42"/>
 <junction x="121.92" y="60.96"/>
-<pinref part="VOUT" gate="1" pin="P"/>
+<pinref part="OUT" gate="1" pin="P"/>
 <junction x="121.92" y="63.5"/>
 <junction x="142.24" y="63.5"/>
@@
 <junction x="20.32" y="81.28"/>
 <junction x="53.34" y="81.28"/>
-<pinref part="VIN" gate="1" pin="P"/>
+<pinref part="IN" gate="1" pin="P"/>
 <wire x1="-15.24" y1="81.28" x2="-2.54" y2="81.28" width="0.1524" layer="91"/>
 <junction x="-15.24" y="81.28"/>
